File: KiCad_p0wer/p0wer.sch (KiCad schematic (older format))
At the start: 4 parts, among them J8 CONN_02X20

Commit message: Replaced wiringPi with pigpio and updated kicad schematic.
Parts:
- removed J8: CONN_02X20, symbol CONN_02X20
- removed Remote1: CONN_02X05, symbol CONN_02X05
- removed U_4066_AB1, U_4066_CD1: 4066, symbol 4066
- added 4066_AB_, 4066_CD_: 4066, symbol 4xxx:4066
- added J8: Conn_02x20_Odd_Even, symbol Connector_Generic:Conn_02x20_Odd_Even
- added REMOTE1: Conn_02x05_Odd_Even, symbol Connector_Generic:Conn_02x05_Odd_Even
Connections:
- wire segments 72 -> 78
- no-connect marks 0 -> 31
Other:
- note added: "2.0"
- note added: "20190927"
- note added: "Rev_2.0 changes:\n- Updated components for compatibility with latest KiCAD\n- Updated pinout numbering for pigpio (replaces wiringpi)"
- note added: "WiringPi C Library Pin References\n----------------\nJ8 | pigpio | Function\n----------------\n29 | 05 | RPI_A_ON\n31 | 06 | RPI_A_OFF\n33 | 13 | RPI_B_ON\n35 | 19 | RPI_B_OFF\n36 | 26 | RPI_C_OFF\n37 | 16 | RPI_C_ON\n38 | 20 | RPI_D_ON\n40 | 21 | RPI_D_OFF"
- note removed: "1.0"
- note removed: "20170602"
- note removed: "WiringPi C Library Pin References\n----------------\nJ8 | WiringPi | Function\n----------------\n29 | 21 | RPI_A_ON\n31 | 22 | RPI_A_OFF\n33 | 23 | RPI_B_ON\n35 | 24 | RPI_B_OFF\n36 | 27 | RPI_C_OFF\n37 | 25 | RPI_C_ON\n38 | 28 | RPI_D_ON\n40 | 29 | RPI_D_OFF"
